File: Hardware/Battery_Emulator/Cell_1.kicad_sch (KiCad schematic)
At the start: 27 parts, among them Q1 IRFB7545PBF, SW1 Jumper, SW2 Jumper, U1 MCP4651T-103E_ST, U2 ISO1640BDR, U6 LM7805_TO220, U7 LM317_TO-220, U8 MCP6001UT-I/OT

Commit message: Update PCB
Made PCB in Kicad
Parts:
- RV? (x2): footprint Potentiometer_THT:Potentiometer_Bourns_PTA3043_Single_Slide -> Connector_PinHeader_2.54mm:PinHeader_1x03_P2.54mm_Vertical
Connections:
- net SCL: no longer U1.2 (SCL), U2.6 (SCL2)
- net SDA: no longer U1.3 (SDA), U2.7 (SDA2)
- new net SCL_ISO: U1.2 (SCL), U2.6 (SCL2)
- new net SDA_ISO: U1.3 (SDA), U2.7 (SDA2)
Changed lines of the file:
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@@
   (junction (at 75.311 108.204) (diameter 0) (color 0 0 0 0)
   )
-  (junction (at 84.836 108.204) (diameter 0) (color 0 0 0 0)
-  )
   (junction (at 91.186 141.224) (diameter 0) (color 0 0 0 0)
   )
@@
   )
   (junction (at 91.186 132.334) (diameter 0) (color 0 0 0 0)
+  )
+  (junction (at 83.312 108.204) (diameter 0) (color 0 0 0 0)
   )
   (junction (at 86.36 66.675) (diameter 0) (color 0 0 0 0)
@@
   )
   (wire (pts (xy 55.626 108.204) (xy 58.166 108.204))
-    (stroke (width 0) (type default))
-  )
-  (wire (pts (xy 88.646 119.634) (xy 92.456 119.634))
+    (stroke (width 1) (type default))
+  )
+  (wire (pts (xy 84.836 119.634) (xy 92.456 119.634))
     (stroke (width 0) (type default))
   )
@@
   )
   (wire (pts (xy 91.186 141.224) (xy 119.126 141.224))
-    (stroke (width 0) (type default))
+    (stroke (width 1) (type default))
   )
   (wire (pts (xy 74.93 80.645) (xy 83.185 80.645))
@@
   )
   (wire (pts (xy 119.126 141.224) (xy 126.746 141.224))
-    (stroke (width 0) (type default))
+    (stroke (width 1) (type default))
   )
   (wire (pts (xy 124.206 165.989) (xy 124.206 162.814))
@@
   )
   (wire (pts (xy 183.261 141.224) (xy 187.706 141.224))
-    (stroke (width 0) (type default))
+    (stroke (width 1) (type default))
   )
   (wire (pts (xy 183.261 119.634) (xy 183.261 108.204))
-    (stroke (width 0) (type default))
+    (stroke (width 1) (type default))
   )
   (wire (pts (xy 183.261 129.794) (xy 183.261 131.064))
-    (stroke (width 0) (type default))
+    (stroke (width 1) (type default))
   )
   (wire (pts (xy 128.016 156.464) (xy 130.556 156.464))
@@
   )
   (wire (pts (xy 35.941 108.204) (xy 40.386 108.204))
-    (stroke (width 0) (type default))
+    (stroke (width 1) (type default))
   )
   (wire (pts (xy 142.621 134.874) (xy 144.526 134.874))
     (stroke (width 0) (type default))
   )
-  (wire (pts (xy 75.311 108.204) (xy 84.836 108.204))
-    (stroke (width 0) (type default))
+  (wire (pts (xy 75.311 108.204) (xy 83.312 108.204))
+    (stroke (width 1) (type default))
   )
   (wire (pts (xy 75.311 128.524) (xy 75.311 141.224))
@@
   )
   (wire (pts (xy 81.28 66.675) (xy 86.36 66.675))
-    (stroke (width 0) (type default))
+    (stroke (width 1) (type default))
   )
   (wire (pts (xy 107.696 162.814) (xy 107.696 165.989))
@@
   )
   (wire (pts (xy 35.941 141.224) (xy 48.006 141.224))
-    (stroke (width 0) (type default))
+    (stroke (width 1) (type default))
   )
   (wire (pts (xy 159.766 127.254) (xy 158.496 127.254))
@@
   )
   (wire (pts (xy 81.28 48.26) (xy 81.28 55.88))
-    (stroke (width 0) (type default))
+    (stroke (width 1) (type default))
   )
   (wire (pts (xy 183.261 131.064) (xy 183.261 132.334))
-    (stroke (width 0) (type default))
+    (stroke (width 1) (type default))
   )
   (wire (pts (xy 88.646 117.094) (xy 92.456 117.094))
@@
   )
   (wire (pts (xy 58.166 141.224) (xy 75.311 141.224))
-    (stroke (width 0) (type default))
+    (stroke (width 1) (type default))
   )
   (wire (pts (xy 107.696 165.989) (xy 124.206 165.989))
@@
     (stroke (width 0) (type default))
   )
-  (wire (pts (xy 84.836 127.254) (xy 84.836 108.204))
+  (wire (pts (xy 83.312 127.254) (xy 83.312 108.204))
     (stroke (width 0) (type default))
   )
@@
   )
   (wire (pts (xy 138.811 141.224) (xy 183.261 141.224))
-    (stroke (width 0) (type default))
+    (stroke (width 1) (type default))
   )
   (wire (pts (xy 137.795 65.405) (xy 137.795 66.675))
@@
     (stroke (width 0) (type default))
   )
-  (wire (pts (xy 92.456 127.254) (xy 84.836 127.254))
+  (wire (pts (xy 92.456 127.254) (xy 83.312 127.254))
     (stroke (width 0) (type default))
   )
@@
   )
   (wire (pts (xy 126.746 141.224) (xy 138.811 141.224))
-    (stroke (width 0) (type default))
+    (stroke (width 1) (type default))
   )
   (wire (pts (xy 37.465 78.105) (xy 46.99 78.105))
@@
     (stroke (width 0) (type default))
   )
-  (wire (pts (xy 88.646 122.174) (xy 92.456 122.174))
+  (wire (pts (xy 84.836 122.174) (xy 92.456 122.174))
     (stroke (width 0) (type default))
   )
@@
   )
   (wire (pts (xy 27.051 108.204) (xy 35.941 108.204))
-    (stroke (width 0) (type default))
+    (stroke (width 1) (type default))
   )
   (wire (pts (xy 117.856 122.174) (xy 121.031 122.174))
@@
   )
   (wire (pts (xy 183.261 139.954) (xy 183.261 141.224))
-    (stroke (width 0) (type default))
+    (stroke (width 1) (type default))
   )
   (wire (pts (xy 97.155 48.26) (xy 97.155 54.61))
@@
   )
   (wire (pts (xy 58.166 108.204) (xy 75.311 108.204))
-    (stroke (width 0) (type default))
+    (stroke (width 1) (type default))
   )
   (wire (pts (xy 81.28 55.88) (xy 71.12 55.88))
-    (stroke (width 0) (type default))
+    (stroke (width 1) (type default))
   )
   (wire (pts (xy 27.94 60.96) (xy 41.91 60.96))
@@
     (stroke (width 0) (type default))
   )
-  (wire (pts (xy 84.836 108.204) (xy 183.261 108.204))
-    (stroke (width 0) (type default))
-  )
   (wire (pts (xy 27.051 141.224) (xy 35.941 141.224))
-    (stroke (width 0) (type default))
+    (stroke (width 1) (type default))
   )
   (wire (pts (xy 183.261 108.204) (xy 187.706 108.204))
-    (stroke (width 0) (type default))
+    (stroke (width 1) (type default))
   )
   (wire (pts (xy 91.186 148.209) (xy 107.696 148.209))
     (stroke (width 0) (type default))
   )
+  (wire (pts (xy 83.312 108.204) (xy 183.261 108.204))
+    (stroke (width 1) (type default))
+  )
   (wire (pts (xy 81.28 60.96) (xy 81.28 66.675))
-    (stroke (width 0) (type default))
+    (stroke (width 1) (type default))
   )
   (wire (pts (xy 58.166 108.204) (xy 58.166 113.919))
@@
     (stroke (width 0) (type default))
   )
+  (wire (pts (xy 83.312 108.204) (xy 84.836 108.204))
+    (stroke (width 0) (type default))
+  )
   (wire (pts (xy 48.006 138.049) (xy 48.006 141.224))
     (stroke (width 0) (type default))
   )
   (wire (pts (xy 81.28 48.26) (xy 86.36 48.26))
-    (stroke (width 0) (type default))
+    (stroke (width 1) (type default))
   )
   (wire (pts (xy 86.36 66.675) (xy 97.155 66.675))
@@
   )
   (wire (pts (xy 75.311 141.224) (xy 91.186 141.224))
-    (stroke (width 0) (type default))
+    (stroke (width 1) (type default))
   )
   (wire (pts (xy 126.746 117.094) (xy 138.811 117.094))
@@
   )
   (wire (pts (xy 71.12 60.96) (xy 81.28 60.96))
-    (stroke (width 0) (type default))
+    (stroke (width 1) (type default))
   )
   (wire (pts (xy 27.94 85.725) (xy 27.94 60.96))
@@
   )
   (wire (pts (xy 48.006 141.224) (xy 58.166 141.224))
-    (stroke (width 0) (type default))
+    (stroke (width 1) (type default))
   )
   (rectangle (start 20.955 46.99) (end 60.96 90.805)
@@
     (effects (font (size 1.27 1.27)) (justify left bottom))
   )
-  (label "SCL" (at 92.456 119.634 180) (fields_autoplaced)
-    (effects (font (size 1.27 1.27)) (justify right bottom))
-  )
   (label "GND_ISO" (at 91.186 165.989 0) (fields_autoplaced)
     (effects (font (size 1.27 1.27)) (justify left bottom))
@@
     (effects (font (size 1.27 1.27)) (justify left bottom))
   )
-  (label "SDA" (at 92.456 122.174 180) (fields_autoplaced)
-    (effects (font (size 1.27 1.27)) (justify right bottom))
-  )
   (label "GND_ISO" (at 71.12 60.96 0) (fields_autoplaced)
     (effects (font (size 1.27 1.27)) (justify left bottom))
   )
-  (label "SDA" (at 74.93 80.645 0) (fields_autoplaced)
+  (label "SDA_ISO" (at 74.93 80.645 0) (fields_autoplaced)
     (effects (font (size 1.27 1.27)) (justify left bottom))
   )
@@
     (effects (font (size 1.27 1.27)) (justify left bottom))
   )
-  (label "SCL" (at 74.93 83.185 0) (fields_autoplaced)
+  (label "SCL_ISO" (at 74.93 83.185 0) (fields_autoplaced)
     (effects (font (size 1.27 1.27)) (justify left bottom))
   )
@@
     (effects (font (size 1.27 1.27)) (justify right bottom))
   )
+  (label "SDA_ISO" (at 92.456 122.174 180) (fields_autoplaced)
+    (effects (font (size 1.27 1.27)) (justify right bottom))
+  )
   (label "+9V_ISO" (at 34.671 108.204 180) (fields_autoplaced)
     (effects (font (size 1.27 1.27)) (justify right bottom))
@@
     (effects (font (size 1.27 1.27)) (justify left bottom))
   )
+  (label "SCL_ISO" (at 92.456 119.634 180) (fields_autoplaced)
+    (effects (font (size 1.27 1.27)) (justify right bottom))
+  )
   (hierarchical_label "+12V" (shape input) (at 27.94 52.07 180) (fields_autoplaced)
     (effects (font (size 1.27 1.27)) (justify right))
@@
       (effects (font (size 1.27 1.27)) (justify right))
     )
-    (property "Footprint" "Potentiometer_THT:Potentiometer_Bourns_PTA3043_Single_Slide" (at 138.811 134.874 0)
+    (property "Footprint" "Connector_PinHeader_2.54mm:PinHeader_1x03_P2.54mm_Vertical" (at 138.811 134.874 0)
       (effects (font (size 1.27 1.27)) hide)
     )
@@
       (effects (font (size 1.27 1.27)) (justify right))
     )
-    (property "Footprint" "Potentiometer_THT:Potentiometer_Bourns_PTA3043_Single_Slide" (at 75.311 124.714 0)
-      (effects (font (size 1.27 1.27)) hide)
-    )
+    (property "Footprint" "Connector_PinHeader_2.54mm:PinHeader_1x03_P2.54mm_Vertical" (at 75.311 124.714 0)
+      (effects (font (size 1.27 1.27)) hide)
+    )

Commit message: Update PCB design
Parts:
- removed U6: LM7805_TO220, Package_TO_SOT_THT:TO-220-3_Vertical, symbol Regulator_Linear:LM7805_TO220
- added U9: KA78M05_TO252, Package_TO_SOT_SMD:TO-252-2, symbol Regulator_Linear:KA78M05_TO252
Connections:
- net +5V_ISO: now also U9.3 (VO)
- net +9V_ISO: now also U9.1 (VI)
- net COUT-: now also U9.2 (GND)
Changed lines of the file:
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@@
     )
   )
-  (symbol (lib_id "Regulator_Linear:LM7805_TO220") (at 107.95 48.26 0) (unit 1)
+  (symbol (lib_id "Regulator_Linear:KA78M05_TO252") (at 107.95 48.26 0) (unit 1)
     (in_bom yes) (on_board yes) (dnp no) (fields_autoplaced)
-    (property "Reference" "U6" (at 107.95 41.91 0)
+    (property "Reference" "U9" (at 107.95 43.3451 0)
       (effects (font (size 1.27 1.27)))
     )
-    (property "Value" "LM7805_TO220" (at 107.95 44.45 0)
+    (property "Value" "KA78M05_TO252" (at 107.95 45.2661 0)
       (effects (font (size 1.27 1.27)))
     )
-    (property "Footprint" "Package_TO_SOT_THT:TO-220-3_Vertical" (at 107.95 42.545 0)
+    (property "Footprint" "Package_TO_SOT_SMD:TO-252-2" (at 107.95 42.545 0)
       (effects (font (size 1.27 1.27) italic) hide)
     )
-    (property "Datasheet" "https://www.onsemi.cn/PowerSolutions/document/MC7800-D.PDF" (at 107.95 49.53 0)
+    (property "Datasheet" "https://www.onsemi.com/pub/Collateral/MC78M00-D.PDF" (at 107.95 49.53 0)
       (effects (font (size 1.27 1.27)) hide)
     )
@@
     (instances
       (project "Battery_Emulator"
+        (path "/bb7641ff-0dfd-4f4a-b3be-57afbbb9fdac"
+          (reference "U9") (unit 1)
+        )
         (path "/bb7641ff-0dfd-4f4a-b3be-57afbbb9fdac/86a0f187-fc20-4f8c-b621-2752c8234446"
-          (reference "U6") (unit 1)
+          (reference "U5") (unit 1)
         )
       )
