File: Hardware/Battery_Emulator_v3/Battery_Emulator_Model_Board/Battery_Emulator_Model_Board.kicad_pcb (KiCad board)
At the start: 2 copper layers, 43 parts, among them J1 Vin, J10 Conn_01x05, J11 Conn_01x05, J12 Conn_01x05, J13 Conn_01x05, J14 Conn_01x05, J15 Conn_01x05, J16 Conn_01x05, J17 Conn_01x05, J2 USB4105-GF-A-060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

Commit message: Hardware Update
Updated the v3 model board PCB layout.
Parts:
- moved J10 307.6 mm to (323.9, 118.9), turned to -90 degrees
- moved J11 289.7 mm to (324.6, 97.0)
- moved J9 278.2 mm to (279.7, 118.9), turned to -90 degrees
- moved J17 261.0 mm to (313.7, 86.3), turned to 90 degrees
- moved J16 230.6 mm to (269.5, 86.3), turned to 90 degrees
- moved J15 200.3 mm to (225.3, 86.3), turned to 90 degrees
- moved J8 195.3 mm to (235.4, 118.9), turned to -90 degrees
- moved J14 170.4 mm to (181.3, 86.3), turned to 90 degrees
- moved J7 170.0 mm to (191.4, 118.9), turned to -90 degrees
- moved J6 146.8 mm to (147.4, 118.9), turned to -90 degrees
- moved J5 126.7 mm to (103.4, 118.9), turned to -90 degrees
- moved J3 112.0 mm to (60.4, 118.9), turned to -90 degrees
- moved J13 87.6 mm to (137.3, 86.3), turned to 90 degrees
- moved J12 66.7 mm to (93.3, 86.3), turned to 90 degrees
- moved TP3 61.0 mm to (77.1, 100.8)
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Routing:
- net +5V: track 27.6 -> 595.8 mm, vias 0 -> 2
- net +12V: track 13.1 -> 527.4 mm, vias 0 -> 12
- net /SCL: track 2.88 -> 480.5 mm, vias 0 -> 1
- net /SDA_cell_8-14: track 0.00 -> 338.0 mm, vias 0 -> 2
- net /SDA_cell_1-7: track 0.00 -> 335.4 mm, vias 0 -> 2
- net /TX: track 0.00 -> 14.7 mm, vias 0 -> 2
- net /RX: track 0.00 -> 12.9 mm, vias 0 -> 2
- net /SDA: track 6.93 -> 13.2 mm, vias 0 -> 2
- net GND: track 7.30 -> 8.62 mm, vias 0 -> 1
- added copper zone on B.Cu, net GND

Commit message: Hardware Update
Finished the Model Board PCB
Parts:
- added TP4: GND, TestPoint:TestPoint_Pad_D2.5mm, F.Cu at (80.8, 100.8)
- moved H4 199.8 mm to (305.2, 113.8)
- moved H3 195.9 mm to (305.2, 94.2)
- moved H2 94.7 mm to (85.0, 113.8)
- moved H1 83.9 mm to (85.0, 94.2)
- moved J12 2.87 mm to (93.3, 89.2)
- moved J13 2.87 mm to (137.3, 89.2)
- moved J14 2.87 mm to (181.3, 89.2)
- moved J15 2.87 mm to (225.3, 89.2)
- moved J16 2.87 mm to (269.5, 89.2)
- moved J17 2.87 mm to (313.7, 89.2)
Routing:
- net +12V: track 527.4 -> 569.1 mm, vias 12 -> 13
- net /SCL: track 480.5 -> 463.3 mm, vias 1 -> 38
- net /SDA_cell_8-14: track 338.0 -> 322.5 mm
- net +5V: track 595.8 -> 610.0 mm, vias 2 -> 6
- net GND: track 8.62 -> 10.9 mm, vias 1 -> 36
- net /SDA_cell_1-7: track 335.4 -> 337.2 mm
Other:
- board outline added: 278.4 x 38.2 mm

Commit message: Hardware update
updated the model board pcb and the cell pcb
Changed lines of the file:
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@@
   (segment (start 71.2 120.2) (end 80.8 110.6) (width 0.3) (layer "B.Cu") (net 7))
   (segment (start 64.6 102.8925) (end 64.6 103.6055) (width 0.3) (layer "F.Cu") (net 8))
-  (segment (start 95.8 107) (end 95.8 105.2) (width 0.3) (layer "F.Cu") (net 8))
   (segment (start 66.15 101.605) (end 66.15 100.805) (width 0.3) (layer "F.Cu") (net 8))
   (segment (start 189 105.2) (end 227.8 105.2) (width 0.3) (layer "F.Cu") (net 8))
   (segment (start 316.4 105.2) (end 319.360953 105.2) (width 0.3) (layer "F.Cu") (net 8))
-  (segment (start 95.805 116.605) (end 95.805 111.205) (width 0.3) (layer "F.Cu") (net 8))
   (segment (start 232.8 91.9495) (end 232.8 96.6505) (width 0.3) (layer "F.Cu") (net 8))
   (segment (start 272 105.2) (end 277 105.2) (width 0.3) (layer "F.Cu") (net 8))
+  (segment (start 95.8 110.8045) (end 95.805 110.8095) (width 0.3) (layer "F.Cu") (net 8))
   (segment (start 232.8 98.1495) (end 232.8 105.2) (width 0.3) (layer "F.Cu") (net 8))
   (segment (start 319.360953 105.2) (end 319.361327 105.199626) (width 0.3) (layer "F.Cu") (net 8))
-  (segment (start 95.805 111.205) (end 95.8 111.2) (width 0.3) (layer "F.Cu") (net 8))
   (segment (start 316.4 115.4) (end 316.4 105.2) (width 0.3) (layer "F.Cu") (net 8))
   (segment (start 321.6 100.119954) (end 321.6 105.2) (width 0.3) (layer "F.Cu") (net 8))
@@
   (segment (start 101 91.9495) (end 101 96.6505) (width 0.3) (layer "F.Cu") (net 8))
   (segment (start 183.6 105.2) (end 189 105.2) (width 0.3) (layer "F.Cu") (net 8))
-  (segment (start 95.83034 107.03034) (end 95.8 107) (width 0.3) (layer "F.Cu") (net 8))
   (segment (start 139.8 109.3055) (end 139.8 105.2) (width 0.3) (layer "F.Cu") (net 8))
-  (segment (start 95.83034 108.757585) (end 95.83034 107.03034) (width 0.3) (layer "F.Cu") (net 8))
   (segment (start 321.570023 97.970069) (end 321.599977 98.000023) (width 0.3) (layer "F.Cu") (net 8))
   (segment (start 227.8 109.3055) (end 227.8 105.2) (width 0.3) (layer "F.Cu") (net 8))
@@
   (segment (start 189 98.1495) (end 189 105.2) (width 0.3) (layer "F.Cu") (net 8))
   (segment (start 321.540023 100.059977) (end 321.6 100.119954) (width 0.3) (layer "F.Cu") (net 8))
+  (segment (start 95.8 109.3055) (end 95.8 105.2) (width 0.3) (layer "F.Cu") (net 8))
   (segment (start 64.8625 102.8925) (end 66.15 101.605) (width 0.3) (layer "F.Cu") (net 8))
   (segment (start 272 116.2505) (end 272 110.8045) (width 0.3) (layer "F.Cu") (net 8))
   (segment (start 145 98.1495) (end 145 105.2) (width 0.3) (layer "F.Cu") (net 8))
+  (segment (start 95.805 110.8095) (end 95.805 116.605) (width 0.3) (layer "F.Cu") (net 8))
   (via (at 189 98.1495) (size 0.8) (drill 0.4) (layers "F.Cu" "B.Cu") (net 8))
   (via (at 321.629977 92.970023) (size 0.8) (drill 0.4) (layers "F.Cu" "B.Cu") (net 8))
@@
   (via (at 277 96.6505) (size 0.8) (drill 0.4) (layers "F.Cu" "B.Cu") (net 8))
   (via (at 183.8 109.3055) (size 0.8) (drill 0.4) (layers "F.Cu" "B.Cu") (net 8))
-  (via (at 95.8 111.2) (size 0.8) (drill 0.4) (layers "F.Cu" "B.Cu") (net 8))
+  (via (at 95.8 110.8045) (size 0.8) (drill 0.4) (layers "F.Cu" "B.Cu") (net 8))
   (via (at 227.8 110.8045) (size 0.8) (drill 0.4) (layers "F.Cu" "B.Cu") (net 8))
   (via (at 321.570023 95.029977) (size 0.8) (drill 0.4) (layers "F.Cu" "B.Cu") (net 8))
@@
   (via (at 277.2 91.9495) (size 0.8) (drill 0.4) (layers "F.Cu" "B.Cu") (net 8))
   (via (at 227.8 109.3055) (size 0.8) (drill 0.4) (layers "F.Cu" "B.Cu") (net 8))
-  (via (at 95.83034 108.757585) (size 0.8) (drill 0.4) (layers "F.Cu" "B.Cu") (net 8))
+  (via (at 95.8 109.3055) (size 0.8) (drill 0.4) (layers "F.Cu" "B.Cu") (net 8))
   (via (at 101 98.1495) (size 0.8) (drill 0.4) (layers "F.Cu" "B.Cu") (net 8))
   (via (at 321.6 105.2) (size 0.8) (drill 0.4) (layers "F.Cu" "B.Cu") (net 8))
@@
   (segment (start 95.805 118.93) (end 95.805 116.605) (width 0.3) (layer "B.Cu") (net 8))
   (segment (start 227.805 116.2555) (end 227.8 116.2505) (width 0.3) (layer "B.Cu") (net 8))
+  (segment (start 95.8 109.3055) (end 95.8 110.8045) (width 0.3) (layer "B.Cu") (net 8))
   (segment (start 100.895 89.175) (end 100.895 91.8445) (width 0.3) (layer "B.Cu") (net 8))
   (segment (start 316.27 118.93) (end 316.27 115.53) (width 0.3) (layer "B.Cu") (net 8))
@@
   (segment (start 272.055 116.3055) (end 272 116.2505) (width 0.3) (layer "B.Cu") (net 8))
   (segment (start 139.8 110.8045) (end 139.8 109.3055) (width 0.3) (layer "B.Cu") (net 8))
-  (segment (start 95.8 111.2) (end 95.8 108.787925) (width 0.3) (layer "B.Cu") (net 8))
   (segment (start 183.805 118.93) (end 183.805 116.2555) (width 0.3) (layer "B.Cu") (net 8))
   (segment (start 321.6 105.2) (end 322.2 104.6) (width 0.3) (layer "B.Cu") (net 8))
@@
   (segment (start 145 96.6505) (end 145 98.1495) (width 0.3) (layer "B.Cu") (net 8))
   (segment (start 272.055 118.93) (end 272.055 116.3055) (width 0.3) (layer "B.Cu") (net 8))
-  (segment (start 95.8 108.787925) (end 95.83034 108.757585) (width 0.3) (layer "B.Cu") (net 8))
   (segment (start 139.805 116.2555) (end 139.8 116.2505) (width 0.3) (layer "B.Cu") (net 8))
   (segment (start 321.629977 92.970023) (end 321.629977 94.970023) (width 0.3) (layer "B.Cu") (net 8))

Commit message: Update battery emulator v3 design
Updated design such that its is parallel with the pins
Parts:
- moved J3 307.7 mm to (368.1, 118.9)
- moved J11 34.3 mm to (358.0, 89.2), turned to 90 degrees
Routing:
- net +5V: track 610.0 -> 696.2 mm
- net +12V: track 569.1 -> 654.7 mm, vias 13 -> 14
- net /SCL: track 463.3 -> 513.5 mm, vias 38 -> 41
- net /SDA_cell_8-14: track 322.5 -> 365.9 mm
- net /SDA_cell_1-7: track 337.2 -> 365.0 mm, vias 2 -> 0
- net GND: track 10.9 -> 15.1 mm, vias 36 -> 51
Other:
- board size 278.4 x 38.2 mm -> 323.6 x 38.2 mm

Commit message: Updated mother board + cell PCB
Made +12V trace on mother board 2mm so it can withstand 2A. Improved routing a bit. Changed pinheader to pinsocket on motherboard and pinsocket to pinheader on cell PCB. Mother board is nearly finished, Cell PCB is not finished.
Parts:
- J10, J11, J12, J13, J14, J15, J16, J17, J3, J5, J6, J7, J8, J9: footprint Connector_PinHeader_2.54mm:PinHeader_1x05_P2.54mm_Horizontal -> Connector_PinSocket_2.54mm:PinSocket_1x05_P2.54mm_Horizontal; moved to B.Cu
- moved H3 42.3 mm to (347.4, 94.4)
- moved H4 42.3 mm to (347.4, 114.0)
- moved J7 32.4 mm to (178.7, 89.2)
- moved J3 32.4 mm to (355.4, 89.2)
- moved J6 32.4 mm to (134.7, 89.2)
- moved J8 32.4 mm to (222.7, 89.2)
- moved J5 32.4 mm to (90.7, 89.2)
- moved J10 32.4 mm to (311.2, 89.2)
- moved J9 32.4 mm to (267.0, 89.2)
- moved J14 30.7 mm to (188.9, 118.9)
- moved J11 30.7 mm to (365.6, 118.9)
- moved J16 30.7 mm to (277.1, 118.9)
- moved J12 30.7 mm to (100.9, 118.9)
- moved J13 30.7 mm to (144.9, 118.9)
- moved J15 30.7 mm to (232.9, 118.9)
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Connections:
- J10 pad 2: +5V -> GND
- J10 pad 3: /SDA_cell_1-7 -> +5V
- J10 pad 4: /SCL -> /SDA_cell_1-7
- J10 pad 5: GND -> /SCL
- J11 pad 2: +5V -> GND
- J11 pad 3: /SDA_cell_8-14 -> +5V
- J11 pad 4: /SCL -> /SDA_cell_8-14
- J11 pad 5: GND -> /SCL
- J12 pad 2: +5V -> GND
- J12 pad 3: /SDA_cell_8-14 -> +5V
- J12 pad 4: /SCL -> /SDA_cell_8-14
- J12 pad 5: GND -> /SCL
- J13 pad 2: +5V -> GND
- J13 pad 3: /SDA_cell_8-14 -> +5V
- J13 pad 4: /SCL -> /SDA_cell_8-14
- J13 pad 5: GND -> /SCL
- J14 pad 2: +5V -> GND
- J14 pad 3: /SDA_cell_8-14 -> +5V
- J14 pad 4: /SCL -> /SDA_cell_8-14
- J14 pad 5: GND -> /SCL
- J15 pad 2: +5V -> GND
- J15 pad 3: /SDA_cell_8-14 -> +5V
- J15 pad 4: /SCL -> /SDA_cell_8-14
- J15 pad 5: GND -> /SCL
- J16 pad 2: +5V -> GND
- J16 pad 3: /SDA_cell_8-14 -> +5V
- J16 pad 4: /SCL -> /SDA_cell_8-14
- J16 pad 5: GND -> /SCL
- J17 pad 2: +5V -> GND
- J17 pad 3: /SDA_cell_8-14 -> +5V
- J17 pad 4: /SCL -> /SDA_cell_8-14
- J17 pad 5: GND -> /SCL
- J3 pad 2: +5V -> GND
- J3 pad 3: /SDA_cell_1-7 -> +5V
- J3 pad 4: /SCL -> /SDA_cell_1-7
- J3 pad 5: GND -> /SCL
- J5 pad 2: +5V -> GND
- J5 pad 3: /SDA_cell_1-7 -> +5V
- J5 pad 4: /SCL -> /SDA_cell_1-7
- J5 pad 5: GND -> /SCL
- J6 pad 2: +5V -> GND
- J6 pad 3: /SDA_cell_1-7 -> +5V
- J6 pad 4: /SCL -> /SDA_cell_1-7
- J6 pad 5: GND -> /SCL
- J7 pad 2: +5V -> GND
- J7 pad 3: /SDA_cell_1-7 -> +5V
- J7 pad 4: /SCL -> /SDA_cell_1-7
- J7 pad 5: GND -> /SCL
- J8 pad 2: +5V -> GND
- J8 pad 3: /SDA_cell_1-7 -> +5V
- J8 pad 4: /SCL -> /SDA_cell_1-7
- J8 pad 5: GND -> /SCL
- J9 pad 2: +5V -> GND
- J9 pad 3: /SDA_cell_1-7 -> +5V
- J9 pad 4: /SCL -> /SDA_cell_1-7
- J9 pad 5: GND -> /SCL
Routing:
- net +12V: track 654.7 -> 689.2 mm, vias 14 -> 0
- net +5V: track 696.2 -> 682.9 mm, vias 6 -> 18
- net /SDA_cell_1-7: track 365.0 -> 357.2 mm
- net /SDA_cell_8-14: track 365.9 -> 368.6 mm, vias 2 -> 0
- net /SCL: track 513.5 -> 515.3 mm, vias 41 -> 42
- net GND: track 15.1 -> 15.2 mm, vias 51 -> 99
Other:
- board size 323.6 x 38.2 mm -> 322.2 x 38.2 mm

Commit message: Updated model board a bit after review
Routing:
- net /SDA_cell_1-7: track 357.2 -> 370.1 mm
- net /SDA_cell_8-14: track 368.6 -> 374.4 mm
- net /SCL: track 515.3 -> 511.4 mm
- net +12V: track 689.2 -> 686.6 mm
- net +5V: track 682.9 -> 684.7 mm
- net GND: vias 99 -> 142

Commit message: Updated Mother board and Cell board
Changed pinout of mother board and cell board such that the pin headers are on the top side. Finished mother board PCB and did DRC check on it.
Parts:
- J10, J11, J12, J13, J14, J15, J16, J17, J3, J5, J6, J7, J8, J9: moved to F.Cu
- moved J3 10.2 mm to (365.6, 89.2)
- moved J7 10.2 mm to (188.9, 89.2)
- moved J5 10.2 mm to (100.9, 89.2)
- moved J16 10.2 mm to (266.9, 119.0)
- moved J13 10.2 mm to (134.7, 118.9)
- moved J14 10.2 mm to (178.7, 118.9)
- moved J15 10.2 mm to (222.7, 118.9)
- moved J6 10.2 mm to (144.9, 89.2)
- moved J8 10.2 mm to (232.9, 89.2)
- moved J12 10.2 mm to (90.7, 118.9)
- moved J9 10.2 mm to (277.1, 89.2)
- moved J10 10.2 mm to (321.4, 89.2)
- moved J11 10.2 mm to (355.4, 118.9)
- moved J17 10.1 mm to (311.2, 118.9)
- moved H4 2.68 mm to (349.7, 112.5)
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Connections:
- J10 pad 1: +12V -> /SCL
- J10 pad 2: GND -> /SDA_cell_1-7
- J10 pad 4: /SDA_cell_1-7 -> GND
- J10 pad 5: /SCL -> +12V
- J11 pad 1: +12V -> /SCL
- J11 pad 2: GND -> /SDA_cell_8-14
- J11 pad 4: /SDA_cell_8-14 -> GND
- J11 pad 5: /SCL -> +12V
- J12 pad 1: +12V -> /SCL
- J12 pad 2: GND -> /SDA_cell_8-14
- J12 pad 4: /SDA_cell_8-14 -> GND
- J12 pad 5: /SCL -> +12V
- J13 pad 1: +12V -> /SCL
- J13 pad 2: GND -> /SDA_cell_8-14
- J13 pad 4: /SDA_cell_8-14 -> GND
- J13 pad 5: /SCL -> +12V
- J14 pad 1: +12V -> /SCL
- J14 pad 2: GND -> /SDA_cell_8-14
- J14 pad 4: /SDA_cell_8-14 -> GND
- J14 pad 5: /SCL -> +12V
- J15 pad 1: +12V -> /SCL
- J15 pad 2: GND -> /SDA_cell_8-14
- J15 pad 4: /SDA_cell_8-14 -> GND
- J15 pad 5: /SCL -> +12V
- J16 pad 1: +12V -> /SCL
- J16 pad 2: GND -> /SDA_cell_8-14
- J16 pad 4: /SDA_cell_8-14 -> GND
- J16 pad 5: /SCL -> +12V
- J17 pad 1: +12V -> /SCL
- J17 pad 2: GND -> /SDA_cell_8-14
- J17 pad 4: /SDA_cell_8-14 -> GND
- J17 pad 5: /SCL -> +12V
- J3 pad 1: +12V -> /SCL
- J3 pad 2: GND -> /SDA_cell_1-7
- J3 pad 4: /SDA_cell_1-7 -> GND
- J3 pad 5: /SCL -> +12V
- J5 pad 1: +12V -> /SCL
- J5 pad 2: GND -> /SDA_cell_1-7
- J5 pad 4: /SDA_cell_1-7 -> GND
- J5 pad 5: /SCL -> +12V
- J6 pad 1: +12V -> /SCL
- J6 pad 2: GND -> /SDA_cell_1-7
- J6 pad 4: /SDA_cell_1-7 -> GND
- J6 pad 5: /SCL -> +12V
- J7 pad 1: +12V -> /SCL
- J7 pad 2: GND -> /SDA_cell_1-7
- J7 pad 4: /SDA_cell_1-7 -> GND
- J7 pad 5: /SCL -> +12V
- J8 pad 1: +12V -> /SCL
- J8 pad 2: GND -> /SDA_cell_1-7
- J8 pad 4: /SDA_cell_1-7 -> GND
- J8 pad 5: /SCL -> +12V
- J9 pad 1: +12V -> /SCL
- J9 pad 2: GND -> /SDA_cell_1-7
- J9 pad 4: /SDA_cell_1-7 -> GND
- J9 pad 5: /SCL -> +12V
Routing:
- net /SDA_cell_8-14: track 374.4 -> 369.9 mm
- net /SDA_cell_1-7: track 370.1 -> 372.3 mm
- net +5V: track 684.7 -> 686.1 mm
- net /SCL: track 511.4 -> 510.3 mm
Other:
- board text added: "JLCJLCJLCJLC"

Commit message: added diode
Parts:
- added D2: 1N4007, Diode_THT:D_DO-41_SOD81_P2.54mm_Vertical_KathodeUp, F.Cu at (55.9, 106.7)
- added H5: MountingHole, MountingHole:MountingHole_3.2mm_M3_Pad_Via, F.Cu at (137.2, 101.6)
- added H6: MountingHole, MountingHole:MountingHole_3.2mm_M3_Pad_Via, F.Cu at (303.5, 101.6)
- added H7: MountingHole, MountingHole:MountingHole_3.2mm_M3_Pad_Via, F.Cu at (215.9, 95.9)
- added H8: MountingHole, MountingHole:MountingHole_3.2mm_M3_Pad_Via, F.Cu at (215.9, 112.4)
- H1, H2, H3, H4: footprint MountingHole:MountingHole_3.2mm_M3 -> MountingHole:MountingHole_3.2mm_M3_Pad_Via
- moved TP1 19.3 mm to (61.0, 120.7)
- moved J1 4.01 mm to (53.3, 111.8)
- moved TP3 2.87 mm to (68.8, 117.6)
- moved TP2 1.39 mm to (50.8, 101.6)
Connections:
- J1 pad 1: +12V -> Net-(D2-A)
Routing:
- net /SDA_cell_8-14: track 369.9 -> 379.3 mm
- net +12V: track 686.8 -> 693.3 mm
- net Net-(D2-A): track 0.00 -> 5.08 mm
- net /SDA_cell_1-7: track 372.3 -> 375.5 mm
- net +5V: track 686.1 -> 683.1 mm
